File: EyeSPI-PiCowbell.kicad_sch (KiCad schematic)
At the start: 20 parts, among them J106 EYE_SPI_DISPLAY_FLIP, J107 Conn_01x01, J108 Conn_01x01, J109 Conn_01x01, U101 Pico

Commit message: Production
Parts:
- U101: footprint RPi_Pico:RPi_Pico_SMD_TH -> MCU_RaspberryPi_and_Boards:RPi_Pico_TH
Connections:
- no-connect marks 19 -> 23
Other:
- title: EYESPI Feather Wing -> EYESPI PiCowbell
Changed lines of the file:
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@@
   (paper "A4")
   (title_block
-    (title "EYESPI Feather Wing")
+    (title "EYESPI PiCowbell")
     (date "2023-01-01")
-    (rev "1.0")
+    (rev "1.0.0")
     (company "Resterampe Berlin")
     (comment 3 "https://creativecommons.org/licenses/by-nc/4.0")
@@
   (no_connect (at 86.995 43.18))
   (no_connect (at 51.435 58.42))
+  (no_connect (at 51.435 33.02))
   (no_connect (at 86.995 33.02))
   (no_connect (at 51.435 50.8))
+  (no_connect (at 51.435 30.48))
   (no_connect (at 51.435 55.88))
   (no_connect (at 71.755 83.82))
@@
   (no_connect (at 51.435 53.34))
   (no_connect (at 69.215 83.82))
+  (no_connect (at 207.645 188.595))
   (no_connect (at 86.995 30.48))
   (no_connect (at 86.995 55.88))
@@
   (no_connect (at 86.995 53.34))
   (no_connect (at 51.435 68.58))
+  (no_connect (at 51.435 38.1))
   (bus_entry (at 106.045 78.74) (size 2.54 2.54)
     (stroke (width 0) (type default) (color 0 0 0 0))
@@
     (property "Reference" "U101" (id 0) (at 69.215 22.225 0))
     (property "Value" "Pico" (id 1) (at 69.215 24.765 0))
-    (property "Footprint" "RPi_Pico:RPi_Pico_SMD_TH" (id 2) (at 69.215 54.61 90)
+    (property "Footprint" "MCU_RaspberryPi_and_Boards:RPi_Pico_TH" (id 2) (at 69.215 54.61 90)
       (effects (font (size 1.27 1.27)) hide)
     )
@@
     )
     (path "/dd9fa880-ba15-407a-a159-dbde5c68fffe"
-      (reference "U101") (unit 1) (value "Pico") (footprint "RPi_Pico:RPi_Pico_SMD_TH")
-    )
-  )
+      (reference "U101") (unit 1) (value "Pico") (footprint "MCU_RaspberryPi_and_Boards:RPi_Pico_TH")
+    )
+  )

Commit message: Closes #1 #2 #3
Parts:
- added J101: StemmaQT, Connector_JST:JST_SH_SM04B-SRSS-TB_1x04-1MP_P1.00mm_Horizontal, symbol Resterampe:StemmaQT
- added SW101: SW_Push, Footprints:Switch_SMD_3.95x2.9mm, symbol Switch:SW_Push
- J106: value EYE_SPI_DISPLAY_FLIP -> EYE_SPI_DISPLAY_TYPE_B; symbol Resterampe:EYE_SPI_DISPLAY_FLIP -> Resterampe:EYE_SPI_DISPLAY_TYPE_B
Connections:
- net +3V3: now also J106.18 (VCC), J101.2 (VCC); no longer J106.1 (VCC)
- net BUSY: now also J106.3 (BUSY/TE); no longer J106.16 (BUSY/TE)
- net EYESPI_GPIO1: now also J106.2 (GPIO1); no longer J106.17 (GPIO1)
- net EYESPI_GPIO2: now also J106.1 (GPIO2); no longer J106.18 (GPIO2)
- net EYESPI_MISO: now also J106.13 (MISO); no longer J106.6 (MISO)
- net EYESPI_MOSI: now also J106.14 (MOSI); no longer J106.5 (MOSI)
- net EYESPI_SCK: now also J106.15 (SCK); no longer J106.4 (SCK)
- net EYESPI_SCL: now also J106.6 (SCL); no longer J106.13 (SCL)
- net EYESPI_SDA: now also J106.5 (SDA); no longer J106.14 (SDA)
- net GND: now also J106.16 (GND), J101.1 (GND), SW101.2; no longer J106.3 (GND)
- net INT: now also J106.4 (INT); no longer J106.15 (INT)
- net LITE: now also J106.17 (BL); no longer J106.2 (BL)
- net SCL: now also J101.3 (SDA)
- net SDA: now also J101.4 (SCL)
- net TFT_DC: now also J106.12 (DC); no longer J106.7 (DC)
- net ~{CARD_CS}: now also J106.9 (~{SD_CS}); no longer J106.10 (~{SD_CS})
- net ~{MEM_CS}: now also J106.8 (~{MEM_CS}); no longer J106.11 (~{MEM_CS})
- net ~{TFT_CS}: now also J106.10 (~{DISP_CS}); no longer J106.9 (~{DISP_CS})
- net ~{TFT_RST}: now also J106.11 (~{RESET}); no longer J106.8 (~{RESET})
- net ~{TS_CS}: now also J106.7 (~{TS_CS}); no longer J106.12 (~{TS_CS})
- net ~{RUN}: now reaches U101.30 (RUN)
- net ~{RUN}: now also SW101.1
- no-connect marks 23 -> 21
Changed lines of the file:
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@@
   (title_block
     (title "EYESPI PiCowbell")
-    (date "2023-01-01")
-    (rev "1.0.0")
+    (date "2023-02-08")
+    (rev "2.0.0")
     (company "Resterampe Berlin")
     (comment 3 "https://creativecommons.org/licenses/by-nc/4.0")
@@
   (no_connect (at 51.435 53.34))
   (no_connect (at 69.215 83.82))
-  (no_connect (at 207.645 188.595))
   (no_connect (at 86.995 30.48))
-  (no_connect (at 86.995 55.88))
   (no_connect (at 51.435 66.04))
   (no_connect (at 86.995 53.34))
@@
     (stroke (width 0) (type default) (color 0 0 0 0))
   )
+  (wire (pts (xy 241.3 135.89) (xy 243.84 135.89))
+    (stroke (width 0) (type default) (color 0 0 0 0))
+  )
   (wire (pts (xy 196.215 29.21) (xy 206.375 29.21))
     (stroke (width 0) (type default) (color 0 0 0 0))
@@
     (stroke (width 0) (type default) (color 0 0 0 0))
   )
+  (wire (pts (xy 220.98 135.89) (xy 231.14 135.89))
+    (stroke (width 0) (type default) (color 0 0 0 0))
+  )
   (wire (pts (xy 99.695 161.925) (xy 99.695 174.625))
     (stroke (width 0) (type default) (color 0 0 0 0))
@@
     (stroke (width 0) (type default) (color 0 0 0 0))
   )
+  (wire (pts (xy 86.995 55.88) (xy 97.155 55.88))
+    (stroke (width 0) (type default) (color 0 0 0 0))
+  )
   (wire (pts (xy 37.465 73.66) (xy 51.435 73.66))
     (stroke (width 0) (type default) (color 0 0 0 0))
@@
     (stroke (width 0) (type default) (color 0 0 0 0))
   )
+  (wire (pts (xy 243.84 135.89) (xy 243.84 140.335))
+    (stroke (width 0) (type default) (color 0 0 0 0))
+  )
   (wire (pts (xy 229.87 36.83) (xy 240.03 36.83))
     (stroke (width 0) (type default) (color 0 0 0 0))
@@
     (stroke (width 0) (type default) (color 0 0 0 0))
   )
+  (wire (pts (xy 243.205 90.17) (xy 243.205 92.71))
+    (stroke (width 0) (type default) (color 0 0 0 0))
+  )
   (wire (pts (xy 86.995 66.04) (xy 97.155 66.04))
     (stroke (width 0) (type default) (color 0 0 0 0))
@@
     (stroke (width 0) (type default) (color 0 0 0 0))
   )
+  (wire (pts (xy 220.98 100.33) (xy 234.315 100.33))
+    (stroke (width 0) (type default) (color 0 0 0 0))
+  )
   (wire (pts (xy 134.62 36.83) (xy 144.78 36.83))
     (stroke (width 0) (type default) (color 0 0 0 0))
@@
     (stroke (width 0) (type default) (color 0 0 0 0))
   )
+  (wire (pts (xy 220.98 102.87) (xy 234.315 102.87))
+    (stroke (width 0) (type default) (color 0 0 0 0))
+  )
   (wire (pts (xy 53.34 143.51) (xy 38.1 143.51))
     (stroke (width 0) (type default) (color 0 0 0 0))
   )
+  (wire (pts (xy 243.205 110.49) (xy 243.205 114.935))
+    (stroke (width 0) (type default) (color 0 0 0 0))
+  )
   (text "General signals" (at 139.7 21.59 0)
     (effects (font (size 1.27 1.27)) (justify left bottom))
@@
     (effects (font (size 1.27 1.27)) (justify left bottom))
   )
+  (label "~{RUN}" (at 220.98 135.89 0)
+    (effects (font (size 1.27 1.27)) (justify left bottom))
+  )
+  (label "SDA" (at 220.98 100.33 0)
+    (effects (font (size 1.27 1.27)) (justify left bottom))
+  )
   (label "EYESPI_MOSI" (at 134.62 52.705 0)
     (effects (font (size 1.27 1.27)) (justify left bottom))
@@
     (effects (font (size 1.27 1.27)) (justify left bottom))
   )
+  (label "~{RUN}" (at 87.63 55.88 0)
+    (effects (font (size 1.27 1.27)) (justify left bottom))
+  )
   (label "~{TFT_RST}" (at 40.64 135.89 0)
     (effects (font (size 1.2446 1.2446)) (justify left bottom))
@@
   )
   (label "TFT_DC" (at 178.435 44.45 0)
+    (effects (font (size 1.27 1.27)) (justify left bottom))
+  )
+  (label "SCL" (at 220.98 102.87 0)
     (effects (font (size 1.27 1.27)) (justify left bottom))
   )
@@
     (pin "2")
   )
-  (symbol (lib_id "Resterampe:EYE_SPI_DISPLAY_FLIP") (at 67.31 140.97 0) (unit 1)
+  (symbol (lib_id "Resterampe:EYE_SPI_DISPLAY_TYPE_B") (at 67.31 140.97 0) (unit 1)
     (in_bom yes) (on_board yes)
     (property "Reference" "J106" (id 0) (at 69.85 170.18 0)
       (effects (font (size 1.9304 1.6408)) (justify left bottom))
     )
-    (property "Value" "EYE_SPI_DISPLAY_FLIP" (id 1) (at 74.93 154.94 90)
+    (property "Value" "EYE_SPI_DISPLAY_TYPE_B" (id 1) (at 74.93 156.21 90)
       (effects (font (size 1.9304 1.6408)) (justify left bottom))
     )
-    (property "Footprint" "Connector_FFC-FPC:Hirose_FH12-18S-0.5SH_1x18-1MP_P0.50mm_Horizontal" (id 2) (at 67.31 140.97 0)
-      (effects (font (size 1.27 1.27)) hide)
-    )
-    (property "Datasheet" "https://learn.adafruit.com/adafruit-eyespi-breakout-board/pinouts" (id 3) (at 67.31 140.97 0)
+    (property "Footprint" "Connector_FFC-FPC:Hirose_FH12-18S-0.5SH_1x18-1MP_P0.50mm_Horizontal" (id 2) (at 67.31 187.96 0)
+      (effects (font (size 1.27 1.27)) hide)
+    )
+    (property "Datasheet" "https://learn.adafruit.com/adafruit-eyespi-breakout-board/pinouts" (id 3) (at 66.04 191.77 0)
       (effects (font (size 1.27 1.27)) hide)
     )
@@
     (pin "MP")
   )
+  (symbol (lib_id "power:GND") (at 243.84 140.335 0) (unit 1)
+    (in_bom yes) (on_board yes) (fields_autoplaced)
+    (property "Reference" "#PWR0111" (id 0) (at 243.84 146.685 0)
+      (effects (font (size 1.27 1.27)) hide)
+    )
+    (property "Value" "GND" (id 1) (at 243.84 145.415 0))
+    (property "Footprint" "" (id 2) (at 243.84 140.335 0)
+      (effects (font (size 1.27 1.27)) hide)
+    )
+    (property "Datasheet" "" (id 3) (at 243.84 140.335 0)
+      (effects (font (size 1.27 1.27)) hide)
+    )
+    (pin "1")
+  )
   (symbol (lib_id "power:GND") (at 100.33 86.36 0) (mirror y) (unit 1)
     (in_bom yes) (on_board yes) (fields_autoplaced)
@@
     (pin "2")
   )
+  (symbol (lib_id "power:+3V3") (at 243.205 90.17 0) (unit 1)
+    (in_bom yes) (on_board yes) (fields_autoplaced)
+    (property "Reference" "#PWR0109" (id 0) (at 243.205 93.98 0)
+      (effects (font (size 1.27 1.27)) hide)
+    )
+    (property "Value" "+3V3" (id 1) (at 243.205 84.455 0))
+    (property "Footprint" "" (id 2) (at 243.205 90.17 0)
+      (effects (font (size 1.27 1.27)) hide)
+    )
+    (property "Datasheet" "" (id 3) (at 243.205 90.17 0)
+      (effects (font (size 1.27 1.27)) hide)
+    )
+    (pin "1")
+  )
   (symbol (lib_id "Jumper:SolderJumper_2_Bridged") (at 192.405 29.21 0) (unit 1)
     (in_bom yes) (on_board yes)
@@
     (pin "2")
   )
+  (symbol (lib_id "Resterampe:StemmaQT") (at 236.855 107.95 0) (unit 1)
+    (in_bom yes) (on_board yes) (fields_autoplaced)
+    (property "Reference" "J101" (id 0) (at 255.27 99.8093 0))
+    (property "Value" "StemmaQT" (id 1) (at 255.27 102.3493 0))
+    (property "Footprint" "Connector_JST:JST_SH_SM04B-SRSS-TB_1x04-1MP_P1.00mm_Horizontal" (id 2) (at 238.125 124.46 0)
+      (effects (font (size 1.27 1.27)) hide)
+    )
+    (property "Datasheet" "https://learn.adafruit.com/introducing-adafruit-stemma-qt/technical-specs" (id 3) (at 236.855 127 0)
+      (effects (font (size 1.27 1.27)) hide)
+    )
+    (property "LCSC" "C160404" (id 4) (at 255.27 104.8893 0))
+    (pin "1")
+    (pin "2")
+    (pin "3")
+    (pin "4")
+    (pin "MP")
+  )
   (symbol (lib_id "Connector_Generic:Conn_01x01") (at 248.285 64.77 0) (unit 1)
     (in_bom yes) (on_board yes) (fields_autoplaced)
@@
     )
     (pin "1")
+  )
+  (symbol (lib_id "Switch:SW_Push") (at 236.22 135.89 0) (unit 1)
+    (in_bom yes) (on_board yes) (fields_autoplaced)
+    (property "Reference" "SW101" (id 0) (at 236.22 128.27 0))
+    (property "Value" "SW_Push" (id 1) (at 236.22 130.81 0))
+    (property "Footprint" "Footprints:Switch_SMD_3.95x2.9mm" (id 2) (at 236.22 130.81 0)
+      (effects (font (size 1.27 1.27)) hide)
+    )
+    (property "Datasheet" "~" (id 3) (at 236.22 130.81 0)
+      (effects (font (size 1.27 1.27)) hide)
+    )
+    (pin "1")
+    (pin "2")
   )
   (symbol (lib_id "power:GND") (at 37.465 86.36 0) (unit 1)
@@
     (pin "1")
   )
+  (symbol (lib_id "power:GND") (at 243.205 114.935 0) (unit 1)
+    (in_bom yes) (on_board yes) (fields_autoplaced)
+    (property "Reference" "#PWR0110" (id 0) (at 243.205 121.285 0)
+      (effects (font (size 1.27 1.27)) hide)
+    )
+    (property "Value" "GND" (id 1) (at 243.205 120.015 0))
+    (property "Footprint" "" (id 2) (at 243.205 114.935 0)
+      (effects (font (size 1.27 1.27)) hide)
+    )
+    (property "Datasheet" "" (id 3) (at 243.205 114.935 0)
+      (effects (font (size 1.27 1.27)) hide)
+    )
+    (pin "1")
+  )
   (sheet_instances
     (path "/" (page "1"))
@@
       (reference "#PWR0108") (unit 1) (value "+3V3") (footprint "")
     )
+    (path "/3c614865-bc12-4490-9931-4eba2dccecd1"
+      (reference "#PWR0109") (unit 1) (value "+3V3") (footprint "")
+    )
+    (path "/fc4daf27-f849-4116-b76c-16432c012c75"
+      (reference "#PWR0110") (unit 1) (value "GND") (footprint "")
+    )
+    (path "/165a3abf-ee10-48ef-983f-eb8b91e54b45"
+      (reference "#PWR0111") (unit 1) (value "GND") (footprint "")
+    )
     (path "/d6bfca6c-b550-4d59-a8ff-920f3566b53c"
       (reference "D101") (unit 1) (value "LED") (footprint "LED_SMD:LED_0603_1608Metric_Pad1.05x0.95mm_HandSolder")
     )
+    (path "/ad66f32e-cffa-420d-8dde-86356b403681"
+      (reference "J101") (unit 1) (value "StemmaQT") (footprint "Connector_JST:JST_SH_SM04B-SRSS-TB_1x04-1MP_P1.00mm_Horizontal")
+    )
     (path "/08eeb292-5bb1-4093-89ce-08ec8a892adb"
-      (reference "J106") (unit 1) (value "EYE_SPI_DISPLAY_FLIP") (footprint "Connector_FFC-FPC:Hirose_FH12-18S-0.5SH_1x18-1MP_P0.50mm_Horizontal")
+      (reference "J106") (unit 1) (value "EYE_SPI_DISPLAY_TYPE_B") (footprint "Connector_FFC-FPC:Hirose_FH12-18S-0.5SH_1x18-1MP_P0.50mm_Horizontal")
     )
     (path "/b94809a9-ed99-4dad-a433-ca0fc388ba07"
@@
       (reference "R101") (unit 1) (value "1K") (footprint "Resistor_SMD:R_0603_1608Metric_Pad0.98x0.95mm_HandSolder")
     )
+    (path "/d24f9435-b18d-4bcb-ad6f-39408d61e5a3"
+      (reference "SW101") (unit 1) (value "SW_Push") (footprint "Footprints:Switch_SMD_3.95x2.9mm")
+    )
     (path "/dd9fa880-ba15-407a-a159-dbde5c68fffe"

Commit message: Production
Parts:
- R101: value 1K -> 330R; LCSC C21190 -> C23138
- SW101: LCSC (none) -> C557591
Changed lines of the file:
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@@
       (effects (font (size 1.27 1.27)) (justify left))
     )
-    (property "Value" "1K" (id 1) (at 101.6 137.7949 0)
+    (property "Value" "330R" (id 1) (at 101.6 137.7949 0)
       (effects (font (size 1.27 1.27)) (justify left))
     )
@@
       (effects (font (size 1.27 1.27)) hide)
     )
-    (property "LCSC" "C21190" (id 4) (at 105.41 139.7 0))
+    (property "LCSC" "C23138" (id 4) (at 105.41 139.7 0))
     (pin "1")
     (pin "2")
@@
   )
   (symbol (lib_id "Switch:SW_Push") (at 236.22 135.89 0) (unit 1)
-    (in_bom yes) (on_board yes) (fields_autoplaced)
+    (in_bom yes) (on_board yes)
     (property "Reference" "SW101" (id 0) (at 236.22 128.27 0))
     (property "Value" "SW_Push" (id 1) (at 236.22 130.81 0))
@@
       (effects (font (size 1.27 1.27)) hide)
     )
-    (property "Datasheet" "~" (id 3) (at 236.22 130.81 0)
-      (effects (font (size 1.27 1.27)) hide)
-    )
+    (property "Datasheet" "https://datasheet.lcsc.com/lcsc/2005221232_SHOU-HAN-TS342A2P-WZ_C557591.pdf" (id 3) (at 236.22 130.81 0)
+      (effects (font (size 1.27 1.27)) hide)
+    )
+    (property "LCSC" "C557591" (id 4) (at 236.22 125.73 0))
     (pin "1")
     (pin "2")
@@
     )
     (path "/57042262-ec7b-4a49-be99-910873b65ad7"
-      (reference "R101") (unit 1) (value "1K") (footprint "Resistor_SMD:R_0603_1608Metric_Pad0.98x0.95mm_HandSolder")
+      (reference "R101") (unit 1) (value "330R") (footprint "Resistor_SMD:R_0603_1608Metric_Pad0.98x0.95mm_HandSolder")
     )
     (path "/d24f9435-b18d-4bcb-ad6f-39408d61e5a3"

Commit message: Closed #4 update to KiCad 7
Parts:
- U101: footprint MCU_RaspberryPi_and_Boards:RPi_Pico_TH -> RPi_Pico:RPi_Pico_SMD_TH
Connections:
- net SCL: now also J101.4 (SCL); no longer J101.3 (SDA)
- net SDA: now also J101.3 (SDA); no longer J101.4 (SCL)
